Commit message: fix: use package uri for zed urdf resources

File: zed_wrapper/urdf/zed_descr.urdf.xacro (robot description, xacro)
@@ -24,5 +24,5 @@
   <xacro:arg name="gnss_y" default="0.0" />
   <xacro:arg name="gnss_z" default="0.0" />
-  <xacro:include filename="$(find zed_wrapper)/urdf/zed_macro.urdf.xacro" />
+  <xacro:include filename="package://zed_wrapper/urdf/zed_macro.urdf.xacro" />
   <xacro:zed_camera name="$(arg camera_name)" model="$(arg camera_model)" custom_baseline="$(arg custom_baseline)" enable_gnss="$(arg enable_gnss)">
 	    <origin xyz="$(arg gnss_x) $(arg gnss_y) $(arg gnss_z)" rpy="0 0 0"/>

File: zed_wrapper/urdf/zed_macro.urdf.xacro (robot description, xacro)
@@ -162,5 +162,5 @@
           <origin xyz="${screw_offset_x} 0 ${screw_offset_z}" rpy="0 0 0"/>
           <geometry>
-            <mesh filename="file://$(find zed_msgs)/meshes/${model}.stl"/>
+            <mesh filename="package://zed_msgs/meshes/${model}.stl"/>
           </geometry>
             <material name="zed_mat">
@@ -171,5 +171,5 @@
           <origin xyz="${screw_offset_x} 0 ${screw_offset_z}" rpy="0 0 0"/>
           <geometry>
-            <mesh filename="file://$(find zed_msgs)/meshes/${model}.stl"/>
+            <mesh filename="package://zed_msgs/meshes/${model}.stl"/>
           </geometry>
         </collision>
@@ -188,5 +188,5 @@
             <origin xyz="0 0 0" rpy="0 0 0"/>
             <geometry>
-              <mesh filename="file://$(find zed_msgs)/meshes/${model}.stl"/>
+              <mesh filename="package://zed_msgs/meshes/${model}.stl"/>
             </geometry>
             <material name="zed_mat">
@@ -197,5 +197,5 @@
             <origin xyz="0 0 0" rpy="0 0 0"/>
             <geometry>
-              <mesh filename="file://$(find zed_msgs)/meshes/${model}.stl"/>
+              <mesh filename="package://zed_msgs/meshes/${model}.stl"/>
             </geometry>
           </collision>
@@ -219,5 +219,5 @@
             <origin xyz="0 0 0" rpy="0 0 0"/>
             <geometry>
-              <mesh filename="file://$(find zed_msgs)/meshes/${model}.stl"/>
+              <mesh filename="package://zed_msgs/meshes/${model}.stl"/>
             </geometry>
             <material name="zed_mat">
@@ -228,5 +228,5 @@
             <origin xyz="0 0 0" rpy="0 0 0"/>
             <geometry>
-              <mesh filename="file://$(find zed_msgs)/meshes/${model}.stl"/>
+              <mesh filename="package://zed_msgs/meshes/${model}.stl"/>
             </geometry>
           </collision>
